File: A2Pico2Lite.kicad_sch (KiCad schematic)
At the start: 14 parts, among them J1 Conn_01x03, J4 Apple2_slot, U1 RPI-Pico2

Commit message: Add files via upload
Parts:
- renumbered JP1 to J2
Changed lines of the file:
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@@
 		(dnp no)
 		(fields_autoplaced yes)
-		(property "Reference" "JP1"
+		(property "Reference" "J2"
 			(at 139.7 58.4199 90)
 			(effects
@@
 			(project ""
 				(path "/eaef1172-3351-417c-bfc4-74a598f141cb"
-					(reference "JP1")
+					(reference "J2")
 					(unit 1)
 				)

Commit message: Add files via upload
Other:
- note added: "GND"
- note added: "GP0"
- note added: "~{IRQ}"
Changed lines of the file:
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@@
+		)
+	)
+	(text "GP0"
+		(exclude_from_sim no)
+		(at 129.032 51.308 0)
+		(effects
+			(font
+				(size 1.27 1.27)
+			)
+		)
+	)
+	(text "GND"
+		(exclude_from_sim no)
+		(at 129.032 46.228 0)
+		(effects
+			(font
+				(size 1.27 1.27)
+			)
+		)
+	)
+	(text "~{IRQ}"
+		(exclude_from_sim no)
+		(at 129.032 48.768 0)
+		(effects
+			(font
+				(size 1.27 1.27)
+			)
 		)
 	)
