File: TH/A2Pico2Lite.kicad_pcb (KiCad board)
At the start: 2 copper layers, 65.5 x 44.1 mm, 65 parts, among them J1 PinHeader_1x03_P2.54mm_Vertic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, J2 SolderJumper-2_P1.3mm_Bridged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, U1 Pico

Commit message: Add files via upload
Parts:
- added R7: 10k, Resistor_THT:R_Axial_DIN0204_L3.6mm_D1.6mm_P5.08mm_Horizontal, F.Cu at (155.1, 116.5)
- added R8: 20k, Resistor_THT:R_Axial_DIN0204_L3.6mm_D1.6mm_P5.08mm_Horizontal, F.Cu at (155.1, 114.4)
- moved D2 2.58 mm to (158.3, 116.0)
- moved D1 2.57 mm to (158.3, 112.9)
- moved R3 2.23 mm to (147.5, 116.5)
- moved R6 2.23 mm to (147.5, 114.4)
- moved R1 2.06 mm to (139.8, 116.5)
- moved R4 2.06 mm to (139.8, 114.4)
- moved R2 2.06 mm to (132.0, 116.5)
- moved R5 2.06 mm to (132.0, 114.3)
Connections:
- U1 pad 30: ~{Reset} -> RUN
Routing:
- net RUN: track 0.00 -> 43.5 mm, vias 0 -> 1
- net ~{Reset}: track 56.5 -> 17.1 mm, vias 2 -> 0
- net D0: track 63.1 -> 55.5 mm, vias 1 -> 2
- net D1: track 62.0 -> 58.9 mm
- net VBUS: track 70.1 -> 72.9 mm
- net 5V: track 23.9 -> 21.4 mm
- net VSYS: track 71.4 -> 74.0 mm
- net 5V-1: track 5.30 -> 2.73 mm
- net ~{IOStb}: track 23.1 -> 25.2 mm
- net ~{IOSel}: track 17.4 -> 15.4 mm
- net A10: track 23.3 -> 24.7 mm
- net PHI0: track 54.5 -> 55.6 mm
- net ~{IOStb}_: track 38.7 -> 39.7 mm
- net D7: track 43.7 -> 44.6 mm
- net A11: track 24.0 -> 23.2 mm
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
Commit message: Add files via upload
Parts:
- renumbered R3 to R1, R1 to R3, R7 to R4, R6 to R5, R5 to R6, R4 to R7
Changed lines of the file:
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@@
 		(descr "Resistor, Axial_DIN0204 series, Axial, Horizontal, pin pitch=5.08mm, 0.167W, length*diameter=3.6*1.6mm^2, http://cdn-reichelt.de/documents/datenblatt/B400/1_4W%23YAG.pdf")
 		(tags "Resistor Axial_DIN0204 series Axial Horizontal pin pitch 5.08mm 0.167W length 3.6mm diameter 1.6mm")
-		(property "Reference" "R7"
+		(property "Reference" "R4"
 			(at 2.54 0 0)
 			(layer "F.SilkS")
@@
 		(descr "Resistor, Axial_DIN0204 series, Axial, Horizontal, pin pitch=5.08mm, 0.167W, length*diameter=3.6*1.6mm^2, http://cdn-reichelt.de/documents/datenblatt/B400/1_4W%23YAG.pdf")
 		(tags "Resistor Axial_DIN0204 series Axial Horizontal pin pitch 5.08mm 0.167W length 3.6mm diameter 1.6mm")
-		(property "Reference" "R5"
+		(property "Reference" "R6"
 			(at 2.54 0 0)
 			(layer "F.SilkS")
@@
 		(descr "Resistor, Axial_DIN0204 series, Axial, Horizontal, pin pitch=5.08mm, 0.167W, length*diameter=3.6*1.6mm^2, http://cdn-reichelt.de/documents/datenblatt/B400/1_4W%23YAG.pdf")
 		(tags "Resistor Axial_DIN0204 series Axial Horizontal pin pitch 5.08mm 0.167W length 3.6mm diameter 1.6mm")
-		(property "Reference" "R6"
+		(property "Reference" "R5"
 			(at 2.54 0 0)
 			(layer "F.SilkS")
@@
 		(descr "Resistor, Axial_DIN0204 series, Axial, Horizontal, pin pitch=5.08mm, 0.167W, length*diameter=3.6*1.6mm^2, http://cdn-reichelt.de/documents/datenblatt/B400/1_4W%23YAG.pdf")
 		(tags "Resistor Axial_DIN0204 series Axial Horizontal pin pitch 5.08mm 0.167W length 3.6mm diameter 1.6mm")
-		(property "Reference" "R4"
+		(property "Reference" "R7"
 			(at 2.54 0 0)
 			(layer "F.SilkS")
@@
 		(descr "Resistor, Axial_DIN0204 series, Axial, Horizontal, pin pitch=5.08mm, 0.167W, length*diameter=3.6*1.6mm^2, http://cdn-reichelt.de/documents/datenblatt/B400/1_4W%23YAG.pdf")
 		(tags "Resistor Axial_DIN0204 series Axial Horizontal pin pitch 5.08mm 0.167W length 3.6mm diameter 1.6mm")
-		(property "Reference" "R3"
+		(property "Reference" "R1"
 			(at 2.54 0 0)
 			(layer "F.SilkS")
@@
 		(descr "Resistor, Axial_DIN0204 series, Axial, Horizontal, pin pitch=5.08mm, 0.167W, length*diameter=3.6*1.6mm^2, http://cdn-reichelt.de/documents/datenblatt/B400/1_4W%23YAG.pdf")
 		(tags "Resistor Axial_DIN0204 series Axial Horizontal pin pitch 5.08mm 0.167W length 3.6mm diameter 1.6mm")
-		(property "Reference" "R1"
+		(property "Reference" "R3"
 			(at 2.54 0 0)
 			(layer "F.SilkS")

Commit message: Add files via upload
Parts:
- renumbered J1 to H1
Other:
- board text added: "A2Pico2Lite (c) 2025 Designed by Ralle Palaveev, https://apple2.co.uk/ Concept by Oliver Schmidt, https://a2retro.de/"
- board text removed: "A2Pico2Lite (c) 2025 Board design by Ralle Palaveev, https://apple2.co.uk/ A2Pico2 concept by Oliver Schmidt, https://a2retro.de/"
Changed lines of the file:
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@@
 		(descr "Through hole straight pin header, 1x03, 2.54mm pitch, single row")
 		(tags "Through hole pin header THT 1x03 2.54mm single row")
-		(property "Reference" "J1"
+		(property "Reference" "H1"
 			(at 0 -2.33 180)
 			(layer "F.SilkS")
@@
 		(layer "Edge.Cuts")
 	)
-	(gr_text "A2Pico2Lite (c) 2025\nBoard design by Ralle Palaveev, https://apple2.co.uk/\nA2Pico2 concept by Oliver Schmidt, https://a2retro.de/\n"
+	(gr_text "A2Pico2Lite (c) 2025\nDesigned by Ralle Palaveev, https://apple2.co.uk/\nConcept by Oliver Schmidt, https://a2retro.de/\n"
 		(at 161.0868 102.5398 0)
 		(layer "B.SilkS")
@@
 	)
 	(segment
-		(start 156.2354 115.3922)
-		(end 156.22715 115.40045)
-		(width 0.2)
-		(layer "B.Cu")
-		(net 33)
-	)
-	(segment
-		(start 125.89065 115.40045)
+		(start 125.9332 115.443)
 		(end 124.64605 114.15585)
 		(width 0.2)
@@
 	)
 	(segment
-		(start 122.7208 114.15585)
-		(end 121.4 115.47665)
+		(start 124.64605 114.15585)
+		(end 122.7208 114.15585)
 		(width 0.2)
 		(layer "B.Cu")
@@
 	)
 	(segment
-		(start 156.22715 115.40045)
-		(end 125.89065 115.40045)
-		(width 0.2)
-		(layer "B.Cu")
-		(net 33)
-	)
-	(segment
 		(start 169.9244 115.52745)
 		(end 169.9244 117.61025)
@@
 	)
 	(segment
-		(start 168.3805 119.15415)
-		(end 168.3805 124.03415)
+		(start 122.7208 114.15585)
+		(end 121.4 115.47665)
 		(width 0.2)
 		(layer "B.Cu")
@@
 	)
 	(segment
-		(start 124.64605 114.15585)
-		(end 122.7208 114.15585)
+		(start 168.3805 119.15415)
+		(end 168.3805 124.03415)
 		(width 0.2)
 		(layer "B.Cu")
@@
 	)
 	(segment
+		(start 156.2354 115.3922)
+		(end 156.1846 115.443)
+		(width 0.2)
+		(layer "B.Cu")
+		(net 33)
+	)
+	(segment
 		(start 169.9244 117.61025)
 		(end 168.3805 119.15415)
 		(width 0.2)
 		(layer "B.Cu")
+		(net 33)
+	)
+	(segment
+		(start 156.1846 115.443)
+		(end 125.9332 115.443)
+		(width 0.2)
+		(layer "B.Cu")

Commit message: Add files via upload
Parts:
- removed R5, R6, R7, R8: 20k, Resistor_THT:R_Axial_DIN0204_L3.6mm_D1.6mm_P5.08mm_Horizontal
- R1, R2, R3, R4: value 10k -> 1k
- moved R1 1.03 mm to (147.5, 115.5)
- moved R3 1.03 mm to (139.8, 115.5)
- moved R4 1.03 mm to (155.1, 115.5)
- moved R2 1.01 mm to (132.0, 115.5)
Routing:
- net ~{IOSel}_: track 40.2 -> 38.4 mm, vias 1 -> 2
- net ~{Reset}: track 17.1 -> 18.2 mm
- net ~{IOStb}_: track 39.7 -> 38.7 mm, vias 2 -> 3
- net RUN: track 43.5 -> 42.5 mm
- net ~{IRQ}: track 63.3 -> 62.5 mm
- net ~{DevSel}_: track 36.7 -> 37.3 mm, vias 1 -> 2
- net GND: vias 38 -> 37

Commit message: Add files via upload
Parts:
- added R5: 20k, Resistor_THT:R_Axial_DIN0204_L3.6mm_D1.6mm_P5.08mm_Horizontal, F.Cu at (147.5, 114.4)
- added R6: 20k, Resistor_THT:R_Axial_DIN0204_L3.6mm_D1.6mm_P5.08mm_Horizontal, F.Cu at (132.0, 114.3)
- added R7: 20k, Resistor_THT:R_Axial_DIN0204_L3.6mm_D1.6mm_P5.08mm_Horizontal, F.Cu at (139.8, 114.4)
- R1, R2, R3, R4: value 1k -> 10k
- moved R1 1.03 mm to (147.5, 116.5)
- moved R3 1.03 mm to (139.8, 116.5)
- moved R4 1.03 mm to (155.1, 116.5)
- moved R2 1.01 mm to (132.0, 116.5)
Routing:
- net ~{IOSel}_: track 38.4 -> 40.2 mm, vias 2 -> 1
- net ~{Reset}: track 18.2 -> 17.1 mm
- net ~{IOStb}_: track 38.7 -> 39.7 mm, vias 3 -> 2
- net RUN: track 42.5 -> 43.5 mm
- net ~{IRQ}: track 62.5 -> 63.3 mm
- net ~{DevSel}_: track 37.3 -> 36.7 mm, vias 2 -> 1
- net GND: vias 37 -> 38

Commit message: Add files via upload
Parts:
- added C3: 220p, Capacitor_THT:C_Disc_D5.0mm_W2.5mm_P5.00mm, F.Cu at (127.0, 114.4)
- added C3: 220p, Capacitor_THT:C_Disc_D5.0mm_W2.5mm_P5.00mm, F.Cu at (142.4, 114.4)
- added C3: 220p, Capacitor_THT:C_Disc_D5.0mm_W2.5mm_P5.00mm, F.Cu at (134.7, 114.4)
- moved R7 2.31 mm to (139.8, 112.0)
- moved R5 2.29 mm to (147.5, 112.1)
- moved R6 2.26 mm to (132.0, 112.1)
- moved R2 0.30 mm to (132.0, 116.8)
- moved R1 0.28 mm to (147.5, 116.8)
- moved R3 0.28 mm to (139.8, 116.8)
- renumbered Fu1 to FU1
Routing:
- net GND: track 6.54 -> 27.1 mm, vias 38 -> 39
- net ~{IOStb}: track 25.2 -> 27.3 mm
- net ~{DevSel}: track 7.68 -> 9.79 mm
- net ~{IOSel}_: track 40.2 -> 42.2 mm
- net ~{IOSel}: track 15.4 -> 17.4 mm
- net D2: track 72.1 -> 73.8 mm
- net D6: track 50.5 -> 52.0 mm
- net A7: track 22.2 -> 23.7 mm
- net D3: track 67.2 -> 68.7 mm
- net D4: track 59.5 -> 60.7 mm
- net A5: track 22.2 -> 23.4 mm
- net A4: track 22.2 -> 23.3 mm
- net A8: track 24.6 -> 23.6 mm
- net A1: track 21.1 -> 22.1 mm
- net ~{DevSel}_: track 36.7 -> 37.6 mm
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Other:
- board text added: "A2Pico2Lite (c) 2026 Designed by Ralle Palaveev, https://apple2.co.uk/ Concept by Oliver Schmidt, https://a2retro.de/"
- board text added: "A2Pico2Lite (c) 2026 by Ralle Palaveev, https://apple2.co.uk/"
- board text removed: "A2Pico2Lite (c) 2025 Designed by Ralle Palaveev, https://apple2.co.uk/ Concept by Oliver Schmidt, https://a2retro.de/"
- board text removed: "A2Pico2Lite (c) 2025 by Ralle Palaveev, https://apple2.co.uk/"

Commit message: Add files via upload
Parts:
- R1, R2, R3: value 10k -> 1k
- R4: value 10k -> 2k
- R5, R6, R7: value 20k -> 2k
- moved G*** 12.4 mm to (177.6, 109.3)
- moved REF** 10.1 mm to (173.1, 108.0)
- moved R4 2.08 mm to (155.1, 114.4)
- moved H1 1.00 mm to (118.9, 114.5)
- moved J2 0.21 mm to (120.1, 111.9)
- renumbered C3 to C2, C3 to C4
Routing:
- net ~{IRQ}: track 63.4 -> 57.1 mm, vias 2 -> 0
- net D2: track 73.8 -> 70.1 mm, vias 3 -> 2
- net ~{IOStb}_: track 40.0 -> 43.6 mm
- net RUN: track 43.5 -> 40.1 mm
- net ~{Reset}: track 17.1 -> 20.1 mm, vias 0 -> 1
- net PHI0: track 56.4 -> 53.8 mm
- net R~{W}: track 54.0 -> 56.3 mm
- net D3: track 68.7 -> 66.8 mm
- net D0: track 55.5 -> 57.3 mm, vias 2 -> 1
- net GPIO0: track 15.3 -> 13.6 mm
- net D4: track 60.7 -> 59.0 mm
- net D5: track 55.6 -> 54.2 mm
- net A7: track 23.7 -> 24.4 mm
- net D1: track 58.9 -> 59.6 mm
- net ~{DevSel}_: track 37.6 -> 37.1 mm
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Other:
- outline, holes or cut-outs redrawn

Commit message: Add files via upload
Routing:
- net ~{DevSel}_: track 37.1 -> 38.8 mm
- net GND: vias 42 -> 43
