File: TH/A2Pico2Lite.kicad_pcb (KiCad board)
At the start: 2 copper layers, 65.5 x 44.1 mm, 69 parts, among them J2 SolderJumper-2_P1.3mm_Bridged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, U1 Pico

Commit message: Add files via upload
Parts:
- removed C2, C3, C4: 220p, Capacitor_THT:C_Disc_D5.0mm_W2.5mm_P5.00mm
- moved R7 1.45 mm to (139.8, 113.5)
- moved R5 1.42 mm to (147.5, 113.5)
- moved R6 1.42 mm to (132.0, 113.5)
- moved R1 1.17 mm to (147.5, 115.6)
- moved R2 1.17 mm to (132.0, 115.6)
- moved R3 1.17 mm to (139.8, 115.6)
Routing:
- net GND: track 27.1 -> 6.54 mm, vias 43 -> 46
- net ~{DevSel}_: track 38.8 -> 35.2 mm
- net ~{IOStb}_: track 43.6 -> 46.1 mm
- net ~{IOSel}_: track 42.9 -> 40.9 mm
- net ~{IOSel}: track 17.6 -> 15.7 mm
- net D7: track 45.3 -> 43.5 mm
- net ~{IOStb}: track 27.5 -> 25.9 mm
- net ~{DevSel}: track 9.82 -> 8.57 mm
- net ~{IRQ}: track 57.0 -> 58.0 mm
- net D3: track 66.4 -> 65.7 mm
- net A4: track 23.4 -> 22.7 mm
- net D4: track 59.0 -> 58.4 mm
- net A5: track 23.4 -> 22.8 mm
- net A10: track 24.7 -> 24.1 mm
