File: TH/A2Pico2Lite.kicad_pcb (KiCad board)
At the start: 2 copper layers, 65.5 x 44.1 mm, 66 parts, among them J2 SolderJumper-2_P1.3mm_Bridged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, U1 Pico

Commit message: Add files via upload
Connections:
- U1 pad 37: 3V3_en -> VSYS
Routing:
- net VSYS: track 74.0 -> 78.7 mm
- net VBUS: track 73.3 -> 74.1 mm, vias 1 -> 2
- net GND: vias 46 -> 47
