File: TH/A2Pico2Lite.kicad_sch (KiCad schematic)
At the start: 14 parts, among them J1 Conn_01x03, J2 SolderJumper_2_Bridged, J4 Apple2_slot, U1 RPI-Pico2

Commit message: Add files via upload
Parts:
- added R4: 10k, Resistor_SMD:R_0402_1005Metric_Pad0.72x0.64mm_HandSolder, symbol Device:R
- added R8: 20k, Resistor_SMD:R_0402_1005Metric_Pad0.72x0.64mm_HandSolder, symbol Device:R
- renumbered J4 to J3, R3 to R1, R1 to R3, R6 to R5, R5 to R6, R4 to R7
Connections:
- net GND: now also R8.1
- net ~{Reset}: now also R4.2; no longer U1.30 (RUN)
- new net: R4.1, R8.2, U1.30 (RUN)
Other:
- moved on the sheet: R1, R2, R3, R5, R6, R7

Commit message: Add files via upload
Parts:
- renumbered J1 to H1, J3 to H2, J2 to J1
Changed lines of the file:
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@@
 		(on_board yes)
 		(dnp no)
-		(property "Reference" "J3"
+		(property "Reference" "H2"
 			(at 96.52 64.77 0)
 			(effects
@@
 			(project "A2Pico.v2.7"
 				(path "/eaef1172-3351-417c-bfc4-74a598f141cb"
-					(reference "J3")
+					(reference "H2")
 					(unit 1)
 				)
@@
 		(dnp no)
 		(fields_autoplaced yes)
-		(property "Reference" "J2"
+		(property "Reference" "J1"
 			(at 139.7 58.4199 90)
 			(effects
@@
 			(project ""
 				(path "/eaef1172-3351-417c-bfc4-74a598f141cb"
-					(reference "J2")
+					(reference "J1")
 					(unit 1)
 				)
@@
 		(dnp no)
 		(fields_autoplaced yes)
-		(property "Reference" "J1"
+		(property "Reference" "H1"
 			(at 120.65 40.64 0)
 			(effects
@@
 			(project ""
 				(path "/eaef1172-3351-417c-bfc4-74a598f141cb"
-					(reference "J1")
+					(reference "H1")
 					(unit 1)
 				)

Commit message: Add files via upload
Parts:
- removed R5, R6, R7, R8: 20k, Resistor_SMD:R_0402_1005Metric_Pad0.72x0.64mm_HandSolder, symbol Device:R

Commit message: Add files via upload
Parts:
- R1, R2, R3, R4: value 10k -> 1k
Changed lines of the file:
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@@
 			)
 		)
-		(property "Value" "10k"
+		(property "Value" "1k"
 			(at 224.79 87.63 90)
 			(effects
@@
 			)
 		)
-		(property "Value" "10k"
+		(property "Value" "1k"
 			(at 231.14 90.17 90)
 			(effects
@@
 			)
 		)
-		(property "Value" "10k"
+		(property "Value" "1k"
 			(at 218.44 85.09 90)
 			(effects
@@
 			)
 		)
-		(property "Value" "10k"
+		(property "Value" "1k"
 			(at 212.09 80.01 90)
 			(effects

Commit message: Add files via upload
Parts:
- added R5, R6, R7: 20k, Resistor_SMD:R_0402_1005Metric_Pad0.72x0.64mm_HandSolder, symbol Device:R
- R1, R2, R3, R4: value 1k -> 10k
Connections:
- net GND: now also R5.1, R6.1, R7.1
- net at R3.1, U1.31 (GP26): now also R7.2
- net at R2.1, U1.32 (GP27): now also R6.2
- net at R1.1, U1.34 (GP28): now also R5.2

Commit message: Add files via upload
Parts:
- added C2, C3, C4: 220p, symbol Device:C
- R1, R2, R3, R4: value 10k -> 1k
- R5, R6, R7: value 20k -> 2k
Connections:
- net ~{DevSel}: now also C4.2
- net ~{IOSel}: now also C3.2
- net ~{IOStb}: now also C2.2
- net at R2.1, R6.2, U1.32 (GP27): now also C3.1
- net at R3.1, R7.2, U1.31 (GP26): now also C4.1
- net at R1.1, R5.2, U1.34 (GP28): now also C2.1
Other:
- moved on the sheet: R2, R3, R4

Commit message: Add files via upload
Parts:
- removed C2, C3, C4: 220p, symbol Device:C
