File: TH/A2Pico2Lite.kicad_sch (KiCad schematic)
At the start: 15 parts, among them J1 SolderJumper_2_Bridged, U1 RPI-Pico2

Commit message: Add files via upload
Connections:
- net at D2.1 (K), U1.39 (VSYS): now also U1.37 (3V3_EN)
Changed lines of the file:
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@@
 	)
 	(junction
+		(at 168.91 60.96)
+		(diameter 0)
+		(color 0 0 0 0)
+	)
+	(junction
 		(at 162.56 137.16)
 		(diameter 0)
@@
 	(wire
 		(pts
+			(xy 173.99 63.5) (xy 171.45 63.5)
+		)
+		(stroke
+			(width 0)
+			(type default)
+		)
+	)
+	(wire
+		(pts
 			(xy 143.51 118.11) (xy 146.05 118.11)
 		)
@@
 	(wire
 		(pts
-			(xy 168.91 63.5) (xy 168.91 54.61)
+			(xy 168.91 60.96) (xy 168.91 54.61)
+		)
+		(stroke
+			(width 0)
+			(type default)
+		)
+	)
+	(wire
+		(pts
+			(xy 168.91 63.5) (xy 168.91 60.96)
 		)
 		(stroke
@@
 	(wire
 		(pts
+			(xy 191.77 60.96) (xy 191.77 72.39)
+		)
+		(stroke
+			(width 0)
+			(type default)
+		)
+	)
+	(wire
+		(pts
 			(xy 167.64 137.16) (xy 165.1 137.16)
 		)
@@
 	(wire
 		(pts
+			(xy 168.91 60.96) (xy 191.77 60.96)
+		)
+		(stroke
+			(width 0)
+			(type default)
+		)
+	)
+	(wire
+		(pts
 			(xy 78.74 78.74) (xy 81.28 78.74)
 		)
@@
 	(symbol
 		(lib_id "power:+3V3")
-		(at 171.45 63.5 270)
+		(at 173.99 63.5 270)
 		(unit 1)
 		(exclude_from_sim no)
@@
 		(dnp no)
 		(property "Reference" "#PWR05"
-			(at 167.64 63.5 0)
+			(at 170.18 63.5 0)
 			(effects
 				(font
@@
 		)
 		(property "Value" "+3V3"
-			(at 177.546 63.5 90)
+			(at 180.086 63.5 90)
 			(effects
 				(font
@@
 		)
 		(property "Footprint" ""
-			(at 171.45 63.5 0)
+			(at 173.99 63.5 0)
 			(effects
 				(font
@@
 		)
 		(property "Datasheet" ""
-			(at 171.45 63.5 0)
+			(at 173.99 63.5 0)
 			(effects
 				(font
@@
 		)
 		(property "Description" ""
-			(at 171.45 63.5 0)
+			(at 173.99 63.5 0)
 			(effects
 				(font
