File: W/A2Pico2LiteW.kicad_pcb (KiCad board)
At the start: 2 copper layers, 65.5 x 44.1 mm, 66 parts, among them J2 SolderJumper-2_P1.3mm_Bridged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, U1 Pico

Commit message: Add files via upload
Parts:
- removed J2: SolderJumper-2_P1.3mm_Bridged_RoundedPad1.0x1.5mm, Jumper:SolderJumper-2_P1.3mm_Bridged_RoundedPad1.0x1.5mm
- removed the R1 at (147.0, 115.6)
- removed R3: 1k, Resistor_SMD:R_0402_1005Metric
- removed R5, R6, R7: 2k, Resistor_SMD:R_0402_1005Metric
- added C2: 100n, Capacitor_SMD:C_0402_1005Metric_Pad0.74x0.62mm_HandSolder, F.Cu at (132.6, 113.5)
- added U2: SN74LVC1G11DBVR, Package_TO_SOT_SMD:SOT-23-6, F.Cu at (129.9, 114.5)
- H1: value PinHeader_1x03_P2.54mm_Vertical -> PinHeader_1x02_P2.54mm_Vertical; footprint Connector_PinHeader_2.54mm:PinHeader_1x03_P2.54mm_Vertical -> Connector_PinHeader_2.54mm:PinHeader_1x02_P2.54mm_Vertical
- R2: value 1k -> 2k
- moved R2 26.2 mm to (153.6, 114.6)
- renumbered R4 to R1
Connections:
- H1 pad 1: GPIO0 -> GND
- H1 pad 2: ~{IRQ} -> Tx
- R1 pad 2: RUN -> ~{Reset_}
- R2 pad 1: ~{IOSel}_ -> GND
- R2 pad 2: ~{IOSel} -> ~{Reset_}
- U1 pad 1: GPIO0 -> ~{IRQ}
- U1 pad 31: ~{DevSel}_ -> ~{Enable}
- U1 pad 32: ~{IOSel}_ -> ~{Reset_}
- U1 pad 34: ~{IOStb}_ -> Tx
Routing:
- net ~{IOStb}_: track 52.0 -> 0.00 mm, vias 3 -> 0
- net ~{Reset_}: track 0.00 -> 49.4 mm, vias 0 -> 4
- net ~{IOSel}_: track 46.5 -> 0.00 mm, vias 4 -> 0
- net RUN: track 44.4 -> 0.00 mm, vias 3 -> 0
- net 3.3V: track 0.00 -> 44.0 mm, vias 0 -> 3
- net ~{DevSel}_: track 40.6 -> 0.00 mm, vias 4 -> 0
- net Tx: track 0.00 -> 33.6 mm
- net ~{Enable}: track 0.00 -> 31.5 mm
- net ~{IOStb}: track 25.9 -> 41.3 mm
- net GPIO0: track 13.6 -> 0.00 mm
- net ~{IRQ}: track 57.9 -> 69.1 mm, vias 0 -> 2
- net ~{DevSel}: track 8.35 -> 18.7 mm
- net D0: track 56.9 -> 60.5 mm, vias 1 -> 3
- net D1: track 59.7 -> 62.8 mm, vias 1 -> 2
- net ~{IOSel}: track 16.0 -> 18.6 mm
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