File: W/A2Pico2LiteW.kicad_pcb (KiCad board)
At the start: 2 copper layers, 65.5 x 44.1 mm, 62 parts, among them U1 Pico, U2 SN74LVC1G11DBVR

Commit message: Add files via upload
Other:
- board text added: "GND Tx"
- board text added: "UART"
- board text removed: "GP0 IRQ GND"

Commit message: Add files via upload
Routing:
- net 3.3V: track 44.0 -> 42.4 mm
- net ~{Reset}: track 19.4 -> 20.2 mm
- net GND: vias 51 -> 57

Commit message: Add files via upload
Connections:
- U1 pad 37: 3V3_en -> VSYS
Routing:
- net VSYS: track 76.5 -> 81.2 mm
- net GND: vias 57 -> 58

Commit message: Add files via upload
Parts:
- added R3: 1k, Resistor_SMD:R_0402_1005Metric, F.Cu at (153.6, 116.7)
Routing:
- net RUN: track 0.00 -> 40.1 mm, vias 0 -> 4
- net GND: track 14.1 -> 17.3 mm, vias 58 -> 57
- net ~{Reset_}: track 49.4 -> 47.6 mm
- net ~{Reset}: track 20.2 -> 19.3 mm

Commit message: Add files via upload
Connections:
- R3 pad 1: GND -> 3.3V
Routing:
- net 3.3V: track 42.4 -> 68.3 mm, vias 3 -> 4
- net GND: track 17.3 -> 12.8 mm, vias 57 -> 56
Changed lines of the file:
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@@
 			(layers "F.Cu" "F.Paste" "F.Mask")
 			(roundrect_rratio 0.25)
-			(net 1 "GND")
+			(net 2 "3.3V")
 			(pintype "passive")
 		)
@@
 	)
 	(segment
-		(start 153.416 118.237)
-		(end 154.1546 117.4984)
-		(width 0.25)
-		(layer "F.Cu")
-		(net 1)
-	)
-	(segment
-		(start 134.4422 112.649)
-		(end 134.4422 111.5568)
-		(width 0.25)
-		(layer "F.Cu")
-		(net 1)
-	)
-	(segment
-		(start 132.6388 114.0801)
-		(end 133.0111 114.0801)
-		(width 0.25)
-		(layer "F.Cu")
-		(net 1)
-	)
-	(segment
-		(start 152.0952 118.237)
-		(end 153.416 118.237)
-		(width 0.25)
-		(layer "F.Cu")
-		(net 1)
-	)
-	(segment
 		(start 118.872 114.4778)
 		(end 119.253 114.0968)
@@
 	)
 	(segment
-		(start 133.0111 114.0801)
-		(end 134.4422 112.649)
+		(start 134.0104 113.0808)
+		(end 133.0111 114.0801)
 		(width 0.25)
 		(layer "F.Cu")
@@
 	)
 	(segment
-		(start 154.1546 117.4984)
-		(end 154.1546 116.713)
+		(start 134.0104 112.776)
+		(end 134.0104 113.0808)
 		(width 0.25)
 		(layer "F.Cu")
@@
 		(net 1)
 	)
+	(segment
+		(start 133.0111 114.0801)
+		(end 132.6388 114.0801)
+		(width 0.25)
+		(layer "F.Cu")
+		(net 1)
+	)
 	(via
 		(at 143.9164 90.424)
@@
 	)
 	(via
-		(at 152.0952 118.237)
-		(size 0.8)
-		(drill 0.4)
-		(layers "F.Cu" "B.Cu")
-		(free yes)
-		(net 1)
-	)
-	(via
 		(at 115.945 101.02665)
 		(size 0.8)
@@
 	)
 	(via
-		(at 134.4422 111.5568)
+		(at 134.0104 112.776)
 		(size 0.8)
 		(drill 0.4)
@@
 	)
 	(segment
+		(start 154.1546 117.4984)
+		(end 154.1546 116.713)
+		(width 0.25)
+		(layer "F.Cu")
+		(net 2)
+	)
+	(segment
 		(start 132.6388 112.2426)
 		(end 132.6388 112.9197)
@@
 	)
 	(segment
+		(start 152.2984 117.7798)
+		(end 153.8732 117.7798)
+		(width 0.25)
+		(layer "F.Cu")
+		(net 2)
+	)
+	(segment
 		(start 127.508 92.202)
 		(end 127.508 86.98515)
@@
 	)
 	(segment
+		(start 153.8732 117.7798)
+		(end 154.1546 117.4984)
+		(width 0.25)
+		(layer "F.Cu")
+		(net 2)
+	)
+	(segment
 		(start 129.8702 113.3657)
 		(end 129.8702 112.3188)
@@
 	)
 	(via
+		(at 152.2984 117.7798)
+		(size 0.8)
+		(drill 0.4)
+		(layers "F.Cu" "B.Cu")
+		(net 2)
+	)
+	(via
 		(at 132.6388 112.2426)
 		(size 0.8)
@@
 	)
 	(segment
+		(start 145.2626 110.7948)
+		(end 134.0866 110.7948)
+		(width 0.3)
+		(layer "B.Cu")
+		(net 2)
+	)
+	(segment
 		(start 132.6388 112.2426)
 		(end 132.5626 112.3188)
@@
 	)
 	(segment
+		(start 134.0866 110.7948)
+		(end 132.6388 112.2426)
+		(width 0.3)
+		(layer "B.Cu")
+		(net 2)
+	)
+	(segment
+		(start 152.2476 117.7798)
+		(end 145.2626 110.7948)
+		(width 0.3)
+		(layer "B.Cu")
+		(net 2)
+	)
+	(segment
 		(start 129.8702 112.3188)
 		(end 124.3076 112.3188)
@@
 	)
 	(segment
+		(start 152.2984 117.7798)
+		(end 152.2476 117.7798)
+		(width 0.3)
+		(layer "B.Cu")
+		(net 2)
+	)
+	(segment
 		(start 118.618 102.92365)
 		(end 118.618 102.47915)
@@
 	)
 	(segment
-		(start 152.2984 116.4844)
-		(end 146.9517 111.1377)
+		(start 152.2984 116.586)
+		(end 146.9517 111.2393)
 		(width 0.2)
 		(layer "B.Cu")
@@
 	)
 	(segment
-		(start 146.9517 111.1377)
-		(end 146.9517 111.0615)
+		(start 142.75095 96.647)
+		(end 149.09505 96.647)
 		(width 0.2)
 		(layer "B.Cu")
@@
 	)
 	(segment
-		(start 142.75095 96.647)
-		(end 149.09505 96.647)
+		(start 146.9517 111.2393)
+		(end 146.9517 111.0615)
 		(width 0.2)
 		(layer "B.Cu")
@@
 	)
 	(segment
-		(start 149.09505 96.647)
-		(end 149.098 96.64405)
+		(start 152.2984 116.7384)
+		(end 152.2984 116.586)
 		(width 0.2)
 		(layer "B.Cu")
@@
 	)
 	(segment
-		(start 152.2984 116.7384)
-		(end 152.2984 116.4844)
+		(start 149.09505 96.647)
+		(end 149.098 96.64405)
 		(width 0.2)
 		(layer "B.Cu")

Commit message: Add files via upload
Routing:
- net GND: vias 56 -> 57
Changed lines of the file:
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@@
+	)
+	(via
+		(at 131.9784 111.0234)
+		(size 0.8)
+		(drill 0.4)
+		(layers "F.Cu" "B.Cu")
+		(free yes)
+		(net 1)
 	)
 	(via

Commit message: Add files via upload
Parts:
- removed the R2 at (153.6, 114.6)
- renumbered R3 to R2
Changed lines of the file:
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@@
 		)
 	)
-	(footprint "Resistor_SMD:R_0402_1005Metric"
-		(layer "F.Cu")
-		(at 153.6446 114.5794 180)
-		(descr "Resistor SMD 0402 (1005 Metric), square (rectangular) end terminal, IPC_7351 nominal, (Body size source: IPC-SM-782 page 72, https://www.pcb-3d.com/wordpress/wp-content/uploads/ipc-sm-782a_amendment_1_and_2.pdf), generated with kicad-footprint-generator")
-		(tags "resistor")
-		(property "Reference" "R2"
-			(at -1.4478 -0.0762 0)
-			(layer "F.SilkS")
-			(effects
-				(font
-					(size 0.5 0.5)
-					(thickness 0.1)
-					(bold yes)
-				)
-			)
-		)
-		(property "Value" "2k"
-			(at 0 1.17 0)
-			(layer "F.Fab")
-			(hide yes)
-			(effects
-				(font
-					(size 1 1)
-					(thickness 0.15)
-				)
-			)
-		)
-		(property "Footprint" ""
-			(at 0 0 0)
-			(layer "F.Fab")
-			(hide yes)
-			(effects
-				(font
-					(size 1.27 1.27)
-					(thickness 0.15)
-				)
-			)
-		)
-		(property "Datasheet" ""
-			(at 0 0 0)
-			(layer "F.Fab")
-			(hide yes)
-			(effects
-				(font
-					(size 1.27 1.27)
-					(thickness 0.15)
-				)
-			)
-		)
-		(property "Description" ""
-			(at 0 0 0)
-			(layer "F.Fab")
-			(hide yes)
-			(effects
-				(font
-					(size 1.27 1.27)
-					(thickness 0.15)
-				)
-			)
-		)
-		(attr smd)
-		(fp_line
-			(start -0.153641 0.38)
-			(end 0.153641 0.38)
-			(stroke
-				(width 0.12)
-				(type solid)
-			)
-			(layer "F.SilkS")
-		)
-		(fp_line
-			(start -0.153641 -0.38)
-			(end 0.153641 -0.38)
-			(stroke
-				(width 0.12)
-				(type solid)
-			)
-			(layer "F.SilkS")
-		)
-		(fp_line
-			(start 0.93 0.47)
-			(end -0.93 0.47)
-			(stroke
-				(width 0.05)
-				(type solid)
-			)
-			(layer "F.CrtYd")
-		)
-		(fp_line
-			(start 0.93 -0.47)
-			(end 0.93 0.47)
-			(stroke
-				(width 0.05)
-				(type solid)
-			)
-			(layer "F.CrtYd")
-		)
-		(fp_line
-			(start -0.93 0.47)
-			(end -0.93 -0.47)
-			(stroke
-				(width 0.05)
-				(type solid)
-			)
-			(layer "F.CrtYd")
-		)
-		(fp_line
-			(start -0.93 -0.47)
-			(end 0.93 -0.47)
-			(stroke
-				(width 0.05)
-				(type solid)
-			)
-			(layer "F.CrtYd")
-		)
-		(fp_line
-			(start 0.525 0.27)
-			(end -0.525 0.27)
-			(stroke
-				(width 0.1)
-				(type solid)
-			)
-			(layer "F.Fab")
-		)
-		(fp_line
-			(start 0.525 -0.27)
-			(end 0.525 0.27)
-			(stroke
-				(width 0.1)
-				(type solid)
-			)
-			(layer "F.Fab")
-		)
-		(fp_line
-			(start -0.525 0.27)
-			(end -0.525 -0.27)
-			(stroke
-				(width 0.1)
-				(type solid)
-			)
-			(layer "F.Fab")
-		)
-		(fp_line
-			(start -0.525 -0.27)
-			(end 0.525 -0.27)
-			(stroke
-				(width 0.1)
-				(type solid)
-			)
-			(layer "F.Fab")
-		)
-		(fp_text user "${REFERENCE}"
-			(at 0 0 0)
-			(layer "F.Fab")
-			(effects
-				(font
-					(size 0.26 0.26)
-					(thickness 0.04)
-				)
-			)
-		)
-		(pad "1" smd roundrect
-			(at -0.51 0 180)
-			(size 0.54 0.64)
-			(layers "F.Cu" "F.Paste" "F.Mask")
-			(roundrect_rratio 0.25)
-			(net 1 "GND")
-			(pintype "passive")
-		)
-		(pad "2" smd roundrect
-			(at 0.51 0 180)
-			(size 0.54 0.64)
-			(layers "F.Cu" "F.Paste" "F.Mask")
-			(roundrect_rratio 0.25)
-			(net 36 "~{Reset_}")
-			(pintype "passive")
-		)
-		(model "${KICAD6_3DMODEL_DIR}/Resistor_SMD.3dshapes/R_0402_1005Metric.wrl"
-			(offset
-				(xyz 0 0 0)
-			)
-			(scale
-				(xyz 1 1 1)
-			)
-			(rotate
-				(xyz 0 0 0)
-			)
-		)
-	)
 	(footprint ""
 		(layer "F.Cu")
@@
 		(descr "Resistor SMD 0402 (1005 Metric), square (rectangular) end terminal, IPC_7351 nominal, (Body size source: IPC-SM-782 page 72, https://www.pcb-3d.com/wordpress/wp-content/uploads/ipc-sm-782a_amendment_1_and_2.pdf), generated with kicad-footprint-generator")
 		(tags "resistor")
-		(property "Reference" "R3"
+		(property "Reference" "R2"
 			(at -1.4224 -0.0762 0)
 			(layer "F.SilkS")
@@
 	)
 	(segment
-		(start 153.1346 114.5794)
-		(end 152.3238 114.5794)
+		(start 150.6347 113.6269)
+		(end 156.718 107.5436)
 		(width 0.2)
 		(layer "F.Cu")
@@
 	)
 	(segment
-		(start 150.6347 113.6269)
-		(end 156.718 107.5436)
+		(start 153.1346 115.5172)
+		(end 152.3238 114.7064)
 		(width 0.2)
 		(layer "F.Cu")
@@
 	(segment
 		(start 153.1346 115.6462)
-		(end 153.1346 114.5794)
+		(end 153.1346 115.5172)
+		(width 0.2)
+		(layer "F.Cu")
+		(net 36)
+	)
+	(segment
+		(start 152.3238 114.7064)
+		(end 152.3238 114.5794)
 		(width 0.2)
 		(layer "F.Cu")
