File: W/A2Pico2LiteW.kicad_sch (KiCad schematic)
At the start: 15 parts, among them J1 SolderJumper_2_Bridged, U1 RPI-Pico2

Commit message: Add files via upload
Parts:
- removed H1: Conn_01x03, symbol Connector_Generic:Conn_01x03
- removed J1: SolderJumper_2_Bridged, symbol Jumper:SolderJumper_2_Bridged
- removed R1, R2, R3: 1k, Resistor_SMD:R_0402_1005Metric_Pad0.72x0.64mm_HandSolder, symbol Device:R
- removed R6, R7: 2k, Resistor_SMD:R_0402_1005Metric_Pad0.72x0.64mm_HandSolder, symbol Device:R
- added C2: 100n, symbol Device:C
- added JH1: Conn_01x02, symbol Connector_Generic:Conn_01x02
- added U2: 74LVC1G11, symbol 74xGxx:74LVC1G11
- renumbered R4 to R1, R5 to R2
Connections:
- net +3V3: now also C2.1, U2.5 (VCC)
- net GND: now also C2.2, JH1.1 (Pin_1), U2.2 (GND)
- net ~{DevSel}: now also U2.1
- net ~{IOSel}: now also U2.6
- net ~{IOStb}: now also U2.3
- net ~{IRQ}: now also U1.1 (GP0)
- net at U1.32 (GP27): now also R1.1, R2.2
- net at U1.31 (GP26): now also U2.4
- net TX: now reaches U1.34 (GP28)
- net TX: now also JH1.2 (Pin_2); no longer R2.2
- net at U1.30 (RUN): no longer R1.1
Other:
- note removed: "GND"
- note removed: "GP0"
- note removed: "~{IRQ}"
- moved on the sheet: R1, R2

Commit message: Add files via upload
Parts:
- U1: value RPI-Pico2 -> RPI-Pico2W
Changed lines of the file:
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@@
 			)
 		)
-		(property "Value" "RPI-Pico2"
+		(property "Value" "RPI-Pico2W"
 			(at 163.83 82.55 0)
 			(effects

Commit message: Add files via upload
Connections:
- net +3V3: now also U1.37 (3V3_EN)
Changed lines of the file:
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@@
 	)
 	(junction
+		(at 191.77 63.5)
+		(diameter 0)
+		(color 0 0 0 0)
+	)
+	(junction
 		(at 209.55 46.99)
 		(diameter 0)
@@
 	(wire
 		(pts
+			(xy 191.77 63.5) (xy 171.45 63.5)
+		)
+		(stroke
+			(width 0)
+			(type default)
+		)
+	)
+	(wire
+		(pts
 			(xy 209.55 46.99) (xy 209.55 54.61)
 		)
@@
 	(wire
 		(pts
+			(xy 194.31 63.5) (xy 191.77 63.5)
+		)
+		(stroke
+			(width 0)
+			(type default)
+		)
+	)
+	(wire
+		(pts
 			(xy 167.64 137.16) (xy 165.1 137.16)
 		)
@@
 	(wire
 		(pts
+			(xy 191.77 63.5) (xy 191.77 72.39)
+		)
+		(stroke
+			(width 0)
+			(type default)
+		)
+	)
+	(wire
+		(pts
 			(xy 78.74 78.74) (xy 81.28 78.74)
 		)
@@
 	(symbol
 		(lib_id "power:+3V3")
-		(at 171.45 63.5 270)
+		(at 194.31 63.5 270)
 		(unit 1)
 		(exclude_from_sim no)
@@
 		(dnp no)
 		(property "Reference" "#PWR05"
-			(at 167.64 63.5 0)
+			(at 190.5 63.5 0)
 			(effects
 				(font
@@
 		)
 		(property "Value" "+3V3"
-			(at 177.546 63.5 90)
+			(at 200.406 63.5 90)
 			(effects
 				(font
@@
 		)
 		(property "Footprint" ""
-			(at 171.45 63.5 0)
+			(at 194.31 63.5 0)
 			(effects
 				(font
@@
 		)
 		(property "Datasheet" ""
-			(at 171.45 63.5 0)
+			(at 194.31 63.5 0)
 			(effects
 				(font
@@
 		)
 		(property "Description" ""
-			(at 171.45 63.5 0)
+			(at 194.31 63.5 0)
 			(effects
 				(font

Commit message: Add files via upload
Connections:
- net +3V3: no longer U1.37 (3V3_EN)
- net at D2.1 (K), U1.39 (VSYS): now also U1.37 (3V3_EN)
Changed lines of the file:
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@@
 	)
 	(junction
+		(at 168.91 60.96)
+		(diameter 0)
+		(color 0 0 0 0)
+	)
+	(junction
 		(at 167.64 137.16)
 		(diameter 0)
@@
 	)
 	(junction
-		(at 191.77 63.5)
-		(diameter 0)
-		(color 0 0 0 0)
-	)
-	(junction
 		(at 209.55 46.99)
 		(diameter 0)
@@
 	(wire
 		(pts
+			(xy 172.72 63.5) (xy 171.45 63.5)
+		)
+		(stroke
+			(width 0)
+			(type default)
+		)
+	)
+	(wire
+		(pts
 			(xy 143.51 80.01) (xy 146.05 80.01)
 		)
@@
 	(wire
 		(pts
+			(xy 168.91 60.96) (xy 168.91 54.61)
+		)
+		(stroke
+			(width 0)
+			(type default)
+		)
+	)
+	(wire
+		(pts
 			(xy 78.74 73.66) (xy 81.28 73.66)
 		)
@@
 	(wire
 		(pts
+			(xy 168.91 60.96) (xy 191.77 60.96)
+		)
+		(stroke
+			(width 0)
+			(type default)
+		)
+	)
+	(wire
+		(pts
 			(xy 78.74 99.06) (xy 81.28 99.06)
 		)
@@
 	(wire
 		(pts
-			(xy 191.77 63.5) (xy 171.45 63.5)
-		)
-		(stroke
-			(width 0)
-			(type default)
-		)
-	)
-	(wire
-		(pts
 			(xy 209.55 46.99) (xy 209.55 54.61)
 		)
@@
 	(wire
 		(pts
-			(xy 168.91 63.5) (xy 168.91 54.61)
+			(xy 168.91 63.5) (xy 168.91 60.96)
 		)
 		(stroke
@@
 	(wire
 		(pts
-			(xy 194.31 63.5) (xy 191.77 63.5)
-		)
-		(stroke
-			(width 0)
-			(type default)
-		)
-	)
-	(wire
-		(pts
 			(xy 167.64 137.16) (xy 165.1 137.16)
 		)
@@
 	(wire
 		(pts
-			(xy 191.77 63.5) (xy 191.77 72.39)
+			(xy 191.77 60.96) (xy 191.77 72.39)
 		)
 		(stroke
@@
 	(symbol
 		(lib_id "power:+3V3")
-		(at 194.31 63.5 270)
+		(at 172.72 63.5 270)
 		(unit 1)
 		(exclude_from_sim no)
@@
 		(dnp no)
 		(property "Reference" "#PWR05"
-			(at 190.5 63.5 0)
+			(at 168.91 63.5 0)
 			(effects
 				(font
@@
 		)
 		(property "Value" "+3V3"
-			(at 200.406 63.5 90)
+			(at 178.816 63.5 90)
 			(effects
 				(font
@@
 		)
 		(property "Footprint" ""
-			(at 194.31 63.5 0)
+			(at 172.72 63.5 0)
 			(effects
 				(font
@@
 		)
 		(property "Datasheet" ""
-			(at 194.31 63.5 0)
+			(at 172.72 63.5 0)
 			(effects
 				(font
@@
 		)
 		(property "Description" ""
-			(at 194.31 63.5 0)
+			(at 172.72 63.5 0)
 			(effects
 				(font

Commit message: Add files via upload
Parts:
- added R3: 1k, Resistor_SMD:R_0402_1005Metric_Pad0.72x0.64mm_HandSolder, symbol Device:R
Connections:
- net GND: now also R3.1
- net at U1.30 (RUN): now also R3.2
Other:
- moved on the sheet: C1, C2, D1, D2, Fu1, H2, JH1, R1, R2, U2

Commit message: Add files via upload
Connections:
- net +3V3: now also R3.1
- net GND: no longer R3.1
Changed lines of the file:
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@@
-	)
-	(junction
-		(at 193.04 105.41)
-		(diameter 0)
-		(color 0 0 0 0)
 	)
 	(junction
@@
 		(pts
 			(xy 123.19 78.74) (xy 125.73 78.74)
-		)
-		(stroke
-			(width 0)
-			(type default)
-		)
-	)
-	(wire
-		(pts
-			(xy 186.69 105.41) (xy 193.04 105.41)
 		)
 		(stroke
@@
 					(unit 1)
 				)
+			)
+		)
+	)
+	(symbol
+		(lib_id "power:+3V3")
+		(at 186.69 105.41 180)
+		(unit 1)
+		(exclude_from_sim no)
+		(in_bom yes)
+		(on_board yes)
+		(dnp no)
+		(property "Reference" "#PWR011"
+			(at 186.69 101.6 0)
+			(effects
+				(font
+					(size 1.27 1.27)
+				)
+				(hide yes)
+			)
+		)
+		(property "Value" "+3V3"
+			(at 186.944 109.728 0)
+			(effects
+				(font
+					(size 1.27 1.27)
+				)
+			)
+		)
+		(property "Footprint" ""
+			(at 186.69 105.41 0)
+			(effects
+				(font
+					(size 1.27 1.27)
+				)
+				(hide yes)
+			)
+		)
+		(property "Datasheet" ""
+			(at 186.69 105.41 0)
+			(effects
+				(font
+					(size 1.27 1.27)
+				)
+				(hide yes)
+			)
+		)
+		(property "Description" ""
+			(at 186.69 105.41 0)
+			(effects
+				(font
+					(size 1.27 1.27)
+				)
+				(hide yes)
+			)
+		)
+		(pin "1"
+		)
+		(instances
+			(project "A2Pico2LiteW"
+				(path "/eaef1172-3351-417c-bfc4-74a598f141cb"
+					(reference "#PWR011")
+					(unit 1)
+				)

Commit message: Add files via upload
Parts:
- R1: value 1k -> 10k
- R2: value 2k -> 20k
Changed lines of the file:
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@@
 			)
 		)
-		(property "Value" "2k"
+		(property "Value" "20k"
 			(at 193.04 100.33 90)
 			(effects
@@
 			)
 		)
-		(property "Value" "1k"
+		(property "Value" "10k"
 			(at 200.66 88.9 90)
 			(effects

Commit message: Add files via upload
Parts:
- removed R2: 20k, Resistor_SMD:R_0402_1005Metric_Pad0.72x0.64mm_HandSolder, symbol Device:R
- R1: value 10k -> 1k
- renumbered R3 to R2
Changed lines of the file:
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@@
 	)
 	(junction
-		(at 193.04 88.9)
-		(diameter 0)
-		(color 0 0 0 0)
-	)
-	(junction
 		(at 137.16 140.97)
 		(diameter 0)
@@
 	(wire
 		(pts
-			(xy 193.04 104.14) (xy 193.04 105.41)
-		)
-		(stroke
-			(width 0)
-			(type default)
-		)
-	)
-	(wire
-		(pts
 			(xy 146.05 50.8) (xy 154.94 50.8)
 		)
@@
 	(wire
 		(pts
-			(xy 171.45 88.9) (xy 193.04 88.9)
-		)
-		(stroke
-			(width 0)
-			(type default)
-		)
-	)
-	(wire
-		(pts
 			(xy 123.19 104.14) (xy 125.73 104.14)
 		)
@@
 	(wire
 		(pts
-			(xy 193.04 88.9) (xy 196.85 88.9)
+			(xy 171.45 88.9) (xy 196.85 88.9)
 		)
 		(stroke
@@
 	(wire
 		(pts
-			(xy 193.04 88.9) (xy 193.04 96.52)
-		)
-		(stroke
-			(width 0)
-			(type default)
-		)
-	)
-	(wire
-		(pts
 			(xy 148.59 67.31) (xy 148.59 64.77)
 		)
@@
 	(symbol
 		(lib_id "Device:R")
-		(at 193.04 100.33 180)
-		(unit 1)
-		(exclude_from_sim no)
-		(in_bom yes)
-		(on_board yes)
-		(dnp no)
-		(property "Reference" "R2"
-			(at 190.5 100.33 90)
-			(effects
-				(font
-					(size 1.27 1.27)
-				)
-			)
-		)
-		(property "Value" "20k"
-			(at 193.04 100.33 90)
-			(effects
-				(font
-					(size 1.27 1.27)
-				)
-			)
-		)
-		(property "Footprint" "Resistor_SMD:R_0402_1005Metric_Pad0.72x0.64mm_HandSolder"
-			(at 194.818 100.33 90)
-			(effects
-				(font
-					(size 1.27 1.27)
-				)
-				(hide yes)
-			)
-		)
-		(property "Datasheet" "~"
-			(at 193.04 100.33 0)
-			(effects
-				(font
-					(size 1.27 1.27)
-				)
-				(hide yes)
-			)
-		)
-		(property "Description" ""
-			(at 193.04 100.33 0)
-			(effects
-				(font
-					(size 1.27 1.27)
-				)
-				(hide yes)
-			)
-		)
-		(pin "1"
-		)
-		(pin "2"
-		)
-		(instances
-			(project "A2Pico2Lite"
-				(path "/eaef1172-3351-417c-bfc4-74a598f141cb"
-					(reference "R2")
-					(unit 1)
-				)
-			)
-		)
-	)
-	(symbol
-		(lib_id "Device:R")
 		(at 200.66 88.9 90)
 		(unit 1)
@@
 		(dnp no)
 		(property "Reference" "R1"
-			(at 205.232 87.63 90)
+			(at 200.66 86.614 90)
 			(effects
 				(font
@@
 			)
 		)
-		(property "Value" "10k"
+		(property "Value" "1k"
 			(at 200.66 88.9 90)
 			(effects
@@
 	)
 	(symbol
-		(lib_id "power:GND")
-		(at 193.04 105.41 0)
-		(unit 1)
-		(exclude_from_sim no)
-		(in_bom yes)
-		(on_board yes)
-		(dnp no)
-		(property "Reference" "#PWR01"
-			(at 193.04 111.76 0)
-			(effects
-				(font
-					(size 1.27 1.27)
-				)
-				(hide yes)
-			)
-		)
-		(property "Value" "GND"
-			(at 193.04 109.474 0)
-			(effects
-				(font
-					(size 1.27 1.27)
-				)
-			)
-		)
-		(property "Footprint" ""
-			(at 193.04 105.41 0)
-			(effects
-				(font
-					(size 1.27 1.27)
-				)
-				(hide yes)
-			)
-		)
-		(property "Datasheet" ""
-			(at 193.04 105.41 0)
-			(effects
-				(font
-					(size 1.27 1.27)
-				)
-				(hide yes)
-			)
-		)
-		(property "Description" ""
-			(at 193.04 105.41 0)
-			(effects
-				(font
-					(size 1.27 1.27)
-				)
-				(hide yes)
-			)
-		)
-		(pin "1"
-		)
-		(instances
-			(project "A2Pico2Lite"
-				(path "/eaef1172-3351-417c-bfc4-74a598f141cb"
-					(reference "#PWR01")
-					(unit 1)
-				)
-			)
-		)
-	)
-	(symbol
 		(lib_id "power:+3V3")
 		(at 152.4 67.31 270)
@@
 		(on_board yes)
 		(dnp no)
-		(property "Reference" "R3"
+		(property "Reference" "R2"
 			(at 183.896 100.33 90)
 			(effects
@@
 			(project "A2Pico2LiteW"
 				(path "/eaef1172-3351-417c-bfc4-74a598f141cb"
-					(reference "R3")
+					(reference "R2")
 					(unit 1)
 				)
